Commit message: fix the xacro namespace

File: unitree_description/xacro/common/contact_sensor.xacro (robot description, xacro)
@@ -1,10 +1,9 @@
 <?xml version="1.0"?>
 <robot xmlns:xacro="http://www.ros.org/wiki/xacro" name="contact">
-    <xacro:macro name="CONTACT" params="link_name prefix ns ">
+    <xacro:macro name="CONTACT" params="link_name prefix">
         <gazebo reference="${link_name}">
             <sensor name="${prefix}_foot_contact" type="contact">
                 <update_rate>1000</update_rate>
                 <plugin name="contactPlugin" filename="libunitreeFootContactPlugin.so">
-                    <robotNamespace>/${ns}</robotNamespace>
                 </plugin>
                 <contact>

File: unitree_description/xacro/common/leg.xacro (robot description, xacro)
@@ -2,8 +2,8 @@
 <robot xmlns:xacro="http://www.ros.org/wiki/xacro">
     <xacro:include filename="$(find unitree_description)/xacro/common/transmission.xacro"/>
-    <xacro:macro name="leg" params="prefix mesh_path mirror mirror_dae front_hind front_hind_dae ns *origin">
+    <xacro:macro name="leg" params="prefix mesh_path mirror mirror_dae front_hind front_hind_dae *origin">
         <joint name="${prefix}_hip_joint" type="revolute">
             <xacro:insert_block name="origin"/>
-            <parent link="${ns}_trunk"/>
+            <parent link="trunk"/>
             <child link="${prefix}_hip"/>
             <axis xyz="1 0 0"/>

File: unitree_description/xacro/robot.xacro (robot description, xacro)
@@ -9,5 +9,5 @@
     <xacro:include filename="$(find unitree_description)/xacro/common/contact_sensor.xacro"/>
     <xacro:property name="mesh_path" value="package://unitree_description/xacro/$(arg robot_type)/meshes"/>
-    <link name="$(arg ns)_base">
+    <link name="base">
         <visual>
             <origin rpy="0 0 0" xyz="0 0 0"/>
@@ -17,10 +17,10 @@
         </visual>
     </link>
-    <joint name="$(arg ns)_floating_base" type="fixed">
+    <joint name="floating_base" type="fixed">
         <origin rpy="0 0 0" xyz="0 0 0"/>
-        <parent link="$(arg ns)_base"/>
-        <child link="$(arg ns)_trunk"/>
+        <parent link="base"/>
+        <child link="trunk"/>
     </joint>
-    <link name="$(arg ns)_trunk">
+    <link name="trunk">
         <visual>
             <origin rpy="0 0 0" xyz="0 0 0"/>
@@ -45,15 +45,15 @@
         </inertial>
     </link>
-    <xacro:IMU connected_to="$(arg ns)_trunk" imu_name="$(arg ns)_imu" xyz="0. 0. 0." rpy="0. 0. 0."/>
-    <xacro:leg prefix="$(arg ns)_FR" mesh_path="${mesh_path}" mirror="-1" mirror_dae= "False" front_hind="1" front_hind_dae="True" ns="$(arg ns)">
+    <xacro:IMU connected_to="trunk" imu_name="imu" xyz="0. 0. 0." rpy="0. 0. 0."/>
+    <xacro:leg prefix="FR" mesh_path="${mesh_path}" mirror="-1" mirror_dae= "False" front_hind="1" front_hind_dae="True">
         <origin rpy="0 0 0" xyz="${leg_offset_x} ${-leg_offset_y} 0"/>
     </xacro:leg>
-    <xacro:leg prefix="$(arg ns)_FL" mesh_path="${mesh_path}"  mirror="1" mirror_dae="True" front_hind="1" front_hind_dae="True" ns="$(arg ns)">
+    <xacro:leg prefix="FL" mesh_path="${mesh_path}"  mirror="1" mirror_dae="True" front_hind="1" front_hind_dae="True">
         <origin rpy="0 0 0" xyz="${leg_offset_x} ${leg_offset_y} 0"/>
     </xacro:leg>
-    <xacro:leg prefix="$(arg ns)_RR" mesh_path="${mesh_path}" mirror="-1" mirror_dae="False" front_hind="-1" front_hind_dae="False" ns="$(arg ns)">
+    <xacro:leg prefix="RR" mesh_path="${mesh_path}" mirror="-1" mirror_dae="False" front_hind="-1" front_hind_dae="False">
         <origin rpy="0 0 0" xyz="${-leg_offset_x} ${-leg_offset_y} 0"/>
     </xacro:leg>
-    <xacro:leg prefix="$(arg ns)_RL" mesh_path="${mesh_path}" mirror="1" mirror_dae="True" front_hind="-1" front_hind_dae="False" ns="$(arg ns)">
+    <xacro:leg prefix="RL" mesh_path="${mesh_path}" mirror="1" mirror_dae="True" front_hind="-1" front_hind_dae="False">
         <origin rpy="0 0 0" xyz="${-leg_offset_x} ${leg_offset_y} 0"/>
     </xacro:leg>
@@ -65,13 +65,13 @@
     </gazebo>
     <!-- Foot contacts. -->
-    <xacro:CONTACT link_name="$(arg ns)_FR_calf" prefix="FR" ns="$(arg ns)"/>
-    <xacro:CONTACT link_name="$(arg ns)_FL_calf" prefix="FL" ns="$(arg ns)"/>
-    <xacro:CONTACT link_name="$(arg ns)_RR_calf" prefix="RR" ns="$(arg ns)"/>
-    <xacro:CONTACT link_name="$(arg ns)_RL_calf" prefix="RL" ns="$(arg ns)"/>
-    <gazebo reference="$(arg ns)_base">
+    <xacro:CONTACT link_name="FR_calf" prefix="FR"/>
+    <xacro:CONTACT link_name="FL_calf" prefix="FL"/>
+    <xacro:CONTACT link_name="RR_calf" prefix="RR"/>
+    <xacro:CONTACT link_name="RL_calf" prefix="RL"/>
+    <gazebo reference="base">
         <material>Gazebo/Green</material>
         <turnGravityOff>false</turnGravityOff>
     </gazebo>
-    <gazebo reference="$(arg ns)_trunk">
+    <gazebo reference="trunk">
         <mu1>0.2</mu1>
         <mu2>0.2</mu2>
