Commit message: fixing the xacro files + clean up

File: unitree_description/xacro/robot.xacro (robot description, xacro)
@@ -3,59 +3,6 @@
     <xacro:arg name="ns" default=""/>
     <xacro:arg name="robot_type" default="aliengo"/>
-    <xacro:include filename="$(find unitree_description)/xacro/$(arg robot_type)/const.xacro"/>
-    <xacro:include filename="$(find unitree_description)/xacro/common/materials.xacro"/>
-    <xacro:include filename="$(find unitree_description)/xacro/common/leg.xacro"/>
-    <xacro:include filename="$(find unitree_description)/xacro/common/imu.xacro"/>
-    <xacro:include filename="$(find unitree_description)/xacro/common/contact_sensor.xacro"/>
-    <xacro:property name="mesh_path" value="package://unitree_description/xacro/$(arg robot_type)/meshes"/>
-    <link name="base">
-        <visual>
-            <origin rpy="0 0 0" xyz="0 0 0"/>
-            <geometry>
-                <box size="0.001 0.001 0.001"/>
-            </geometry>
-        </visual>
-    </link>
-    <joint name="floating_base" type="fixed">
-        <origin rpy="0 0 0" xyz="0 0 0"/>
-        <parent link="base"/>
-        <child link="trunk"/>
-    </joint>
-    <link name="trunk">
-        <visual>
-            <origin rpy="0 0 0" xyz="0 0 0"/>
-            <geometry>
-                <mesh filename="${mesh_path}/trunk.dae" scale="1 1 1"/>
-            </geometry>
-            <material name="orange"/>
-        </visual>
-        <collision>
-            <origin rpy="0 0 0" xyz="0 0 0"/>
-            <geometry>
-                <box size="${trunk_length} ${trunk_width} ${trunk_height}"/>
-            </geometry>
-        </collision>
-        <inertial>
-            <origin rpy="0 0 0" xyz="${trunk_com_x} ${trunk_com_y} ${trunk_com_z}"/>
-            <mass value="${trunk_mass}"/>
-            <inertia
-                ixx="${trunk_ixx}" ixy="${trunk_ixy}" ixz="${trunk_ixz}"
-                iyy="${trunk_iyy}" iyz="${trunk_iyz}"
-                izz="${trunk_izz}"/>
-        </inertial>
-    </link>
-    <xacro:IMU connected_to="trunk" imu_name="imu" xyz="0. 0. 0." rpy="0. 0. 0."/>
-    <xacro:leg prefix="FR" mesh_path="${mesh_path}" mirror="-1" mirror_dae= "False" front_hind="1" front_hind_dae="True">
-        <origin rpy="0 0 0" xyz="${leg_offset_x} ${-leg_offset_y} 0"/>
-    </xacro:leg>
-    <xacro:leg prefix="FL" mesh_path="${mesh_path}"  mirror="1" mirror_dae="True" front_hind="1" front_hind_dae="True">
-        <origin rpy="0 0 0" xyz="${leg_offset_x} ${leg_offset_y} 0"/>
-    </xacro:leg>
-    <xacro:leg prefix="RR" mesh_path="${mesh_path}" mirror="-1" mirror_dae="False" front_hind="-1" front_hind_dae="False">
-        <origin rpy="0 0 0" xyz="${-leg_offset_x} ${-leg_offset_y} 0"/>
-    </xacro:leg>
-    <xacro:leg prefix="RL" mesh_path="${mesh_path}" mirror="1" mirror_dae="True" front_hind="-1" front_hind_dae="False">
-        <origin rpy="0 0 0" xyz="${-leg_offset_x} ${leg_offset_y} 0"/>
-    </xacro:leg>
+    <xacro:include filename="$(find unitree_description)/xacro/$(arg robot_type).xacro"/>
+    <xacro:include filename="$(find unitree_description)/xacro/gazebo.xacro"/>
     <gazebo>
         <plugin name="gazebo_ros_control" filename="libgazebo_ros_control.so">
@@ -64,18 +11,3 @@
         </plugin>
     </gazebo>
-    <!-- Foot contacts. -->
-    <xacro:CONTACT link_name="FR_calf" prefix="FR"/>
-    <xacro:CONTACT link_name="FL_calf" prefix="FL"/>
-    <xacro:CONTACT link_name="RR_calf" prefix="RR"/>
-    <xacro:CONTACT link_name="RL_calf" prefix="RL"/>
-    <gazebo reference="base">
-        <material>Gazebo/Green</material>
-        <turnGravityOff>false</turnGravityOff>
-    </gazebo>
-    <gazebo reference="trunk">
-        <mu1>0.2</mu1>
-        <mu2>0.2</mu2>
-        <kp  value="1000000.0"/>
-        <kd  value="1.0"/>
-    </gazebo>
 </robot>
