Commit message: minor update

File: unitree_description/xacro/go1.xacro (robot description, xacro)
@@ -4,6 +4,4 @@
     <xacro:include filename="$(find go1_description)/xacro/materials.xacro"/>
     <xacro:include filename="$(find go1_description)/xacro/leg.xacro"/>
-    <xacro:include filename="$(find go1_description)/xacro/depthCamera.xacro"/>
-    <xacro:include filename="$(find go1_description)/xacro/ultraSound.xacro"/>
     <link name="base">
         <visual>
@@ -71,41 +69,3 @@
     <xacro:leg name="RR" mirror="-1" mirror_dae="False"  front_hind="-1" front_hind_dae="False" />
     <xacro:leg name="RL" mirror="1"  mirror_dae="True"   front_hind="-1" front_hind_dae="False" />
-    <xacro:depthCamera camID="1" name="face">
-        <origin rpy="${PI} 0 0" xyz="0.2785 0.0125 0.0167"/>
-    </xacro:depthCamera>
-    <xacro:depthCamera camID="2" name="chin">
-        <origin rpy="${PI} ${PI/2} 0" xyz="0.2522 0.0125 -0.0436"/>
-    </xacro:depthCamera>
-    <xacro:depthCamera camID="3" name="left">
-        <origin rpy="${PI} 0.2618 ${PI/2}" xyz="-0.066 0.082 -0.0176"/>
-    </xacro:depthCamera>
-    <xacro:depthCamera camID="4" name="right">
-        <origin rpy="${PI} 0.2618 ${-PI/2}" xyz="-0.041 -0.082 -0.0176"/>
-    </xacro:depthCamera>
-    <xacro:depthCamera camID="5" name="rearDown">
-        <origin rpy="${PI} ${PI/2} 0" xyz="-0.0825 0.0125 -0.04365"/>
-    </xacro:depthCamera>
-    <joint name="camera_laserscan_joint_left" type="fixed">
-        <origin rpy="0 0.2618 0" xyz="0 0 0"/>
-        <parent link="camera_left"/>
-        <child link="camera_laserscan_link_left"/>
-    </joint>
-    <link name="camera_laserscan_link_left">
-    </link>
-    <joint name="camera_laserscan_joint_right" type="fixed">
-        <origin rpy="0 0.2618 0" xyz="0 0 0"/>
-        <parent link="camera_right"/>
-        <child link="camera_laserscan_link_right"/>
-    </joint>
-    <link name="camera_laserscan_link_right">
-    </link>
-    <xacro:ultraSound name="left">
-        <origin rpy="0 0.2618 ${PI/2}" xyz="-0.0535  0.0826 0.00868"/>
-    </xacro:ultraSound>
-    <xacro:ultraSound name="right">
-        <origin rpy="0 0.2618 ${-PI/2}" xyz="-0.0535 -0.0826 0.00868"/>
-    </xacro:ultraSound>
-    <xacro:ultraSound name="face">
-        <origin rpy="0 0 0" xyz="0.2747 0.0 -0.0088"/>
-    </xacro:ultraSound>
 </robot>

Commit message: edit go1 xacro

File: unitree_description/xacro/go1.xacro (robot description, xacro)
@@ -4,4 +4,6 @@
     <xacro:include filename="$(find go1_description)/xacro/materials.xacro"/>
     <xacro:include filename="$(find go1_description)/xacro/leg.xacro"/>
+    <xacro:include filename="$(find go1_description)/xacro/depthCamera.xacro"/>
+    <xacro:include filename="$(find go1_description)/xacro/ultraSound.xacro"/>
     <link name="base">
         <visual>
@@ -69,3 +71,41 @@
     <xacro:leg name="RR" mirror="-1" mirror_dae="False"  front_hind="-1" front_hind_dae="False" />
     <xacro:leg name="RL" mirror="1"  mirror_dae="True"   front_hind="-1" front_hind_dae="False" />
+    <xacro:depthCamera camID="1" name="face">
+        <origin rpy="${PI} 0 0" xyz="0.2785 0.0125 0.0167"/>
+    </xacro:depthCamera>
+    <xacro:depthCamera camID="2" name="chin">
+        <origin rpy="${PI} ${PI/2} 0" xyz="0.2522 0.0125 -0.0436"/>
+    </xacro:depthCamera>
+    <xacro:depthCamera camID="3" name="left">
+        <origin rpy="${PI} 0.2618 ${PI/2}" xyz="-0.066 0.082 -0.0176"/>
+    </xacro:depthCamera>
+    <xacro:depthCamera camID="4" name="right">
+        <origin rpy="${PI} 0.2618 ${-PI/2}" xyz="-0.041 -0.082 -0.0176"/>
+    </xacro:depthCamera>
+    <xacro:depthCamera camID="5" name="rearDown">
+        <origin rpy="${PI} ${PI/2} 0" xyz="-0.0825 0.0125 -0.04365"/>
+    </xacro:depthCamera>
+    <joint name="camera_laserscan_joint_left" type="fixed">
+        <origin rpy="0 0.2618 0" xyz="0 0 0"/>
+        <parent link="camera_left"/>
+        <child link="camera_laserscan_link_left"/>
+    </joint>
+    <link name="camera_laserscan_link_left">
+    </link>
+    <joint name="camera_laserscan_joint_right" type="fixed">
+        <origin rpy="0 0.2618 0" xyz="0 0 0"/>
+        <parent link="camera_right"/>
+        <child link="camera_laserscan_link_right"/>
+    </joint>
+    <link name="camera_laserscan_link_right">
+    </link>
+    <xacro:ultraSound name="left">
+        <origin rpy="0 0.2618 ${PI/2}" xyz="-0.0535  0.0826 0.00868"/>
+    </xacro:ultraSound>
+    <xacro:ultraSound name="right">
+        <origin rpy="0 0.2618 ${-PI/2}" xyz="-0.0535 -0.0826 0.00868"/>
+    </xacro:ultraSound>
+    <xacro:ultraSound name="face">
+        <origin rpy="0 0 0" xyz="0.2747 0.0 -0.0088"/>
+    </xacro:ultraSound>
 </robot>
